File: tiny_stick.kicad_pcb (KiCad board)
At the start: 2 copper layers, 61 x 39.8 mm, 31 parts, among them J1 In, J2 Out, J3 Vin, J4 pwr sel, SW1 batt_switch, SW2 SW_Push, U2 AMS1117-5.0

Commit message: Updated with production files
Parts:
- removed the REF** at (130.2, 67.9)
- removed the REF** at (98.4, 67.9)
- added REF**: MountingHole_2.2mm_M2, MountingHole:MountingHole_2.2mm_M2, F.Cu at (97.8, 67.9)
- added REF**: MountingHole_2.2mm_M2, MountingHole:MountingHole_2.2mm_M2, F.Cu at (129.5, 67.9)
- C9: value C -> CP1; footprint Capacitor_Tantalum_SMD:CP_EIA-3528-12_Kemet-T -> Capacitor_Tantalum_SMD:CP_EIA-3528-21_Kemet-B
- moved C9 0.77 mm to (110.2, 97.9)
- moved G*** 0.27 mm to (116.1, 68.8)
- renumbered Tiny85 to U1
Routing:
- net +5V: track 211.1 -> 214.6 mm
- net Net-(C9-Pad1): track 20.3 -> 21.3 mm
