File: tiny_stick.sch (KiCad schematic (older format))
At the start: 28 parts, among them J1 In, J2 Out, J3 Vin, J4 pwr sel, SW1 batt_switch, SW2 SW_Push, U1 ATtiny85-20PU, U2 AMS1117-5.0

Commit message: Updated with production files
Parts:
- removed C9: C, Capacitor_Tantalum_SMD:CP_EIA-3528-12_Kemet-T, symbol Device:C
- added C9: CP1, Capacitor_Tantalum_SMD:CP_EIA-3528-21_Kemet-B, symbol Device:CP1
Connections:
- net GND: now also C9.2
- net at J4.1 (Pin_1), U2.2 (VO): now also C9.1
Changed lines of the file:
@@
 $EndComp
-$Comp
-L Device:C C9
-U 1 1 5E2CB53E
-P 3900 5950
-F 0 "C9" H 4015 5996 50  0000 L CNN
-F 1 "C" H 4015 5905 50  0000 L CNN
-F 2 "Capacitor_Tantalum_SMD:CP_EIA-3528-12_Kemet-T" H 3938 5800 50  0001 C CNN
-F 3 "~" H 3900 5950 50  0001 C CNN
-	1    3900 5950
-	1    0    0    -1
-$EndComp
-Wire Wire Line
-	3600 5800 3900 5800
-Connection ~ 3900 5800
 $Comp
 L power:GND #PWR017
@@
 	4700 5500 4900 5500
 Wire Wire Line
+	3600 5800 3900 5800
+$Comp
+L Device:CP1 C9
+U 1 1 5E307CF7
+P 3900 5950
+F 0 "C9" H 4015 5996 50  0000 L CNN
+F 1 "CP1" H 4015 5905 50  0000 L CNN
+F 2 "Capacitor_Tantalum_SMD:CP_EIA-3528-21_Kemet-B" H 3900 5950 50  0001 C CNN
+F 3 "~" H 3900 5950 50  0001 C CNN
+	1    3900 5950
+	1    0    0    -1
+$EndComp
+Connection ~ 3900 5800
+Wire Wire Line
 	3900 5800 5450 5800
